File: poe_pd_iface.kicad_sch (KiCad schematic)
At the start: 11 parts, among them U2 NCP1090, U3 PG02S4803A

Commit message: Add LCSC part numbers
Parts:
- D1, D2: LCSC (none) -> C895500
- U2: LCSC (none) -> C897681
