File: poe_pd_iface.kicad_sch (KiCad schematic)
At the start: 11 parts, among them U2 NCP1090, U3 PG02S4803A

Commit message: Add LCSC part numbers
Parts:
- C6: LCSC (none) -> CC0805KRX7R9BB104
- C7: LCSC (none) -> C540963
- C8: LCSC (none) -> CL21A106KAYNNNE
- D1, D2: LCSC (none) -> C895500; digikey MDB6SFSCT-ND -> (none)
- D3: LCSC (none) -> C280379
- R5: LCSC (none) -> C321809
- R6: LCSC (none) -> C185366
- R7: LCSC (none) -> C218055
- U2: LCSC (none) -> C897681
- U3: digikey 941-1186-ND -> (none)
