File: w5500_eth_iface.kicad_sch (KiCad schematic)
At the start: 13 parts, among them U4 W5500, Y1 25MHz

Commit message: Add LCSC part numbers
Parts:
- C10, C11, C9: LCSC (none) -> C14663
- C12: LCSC (none) -> C57112
- C13: LCSC (none) -> CL10A475KO8NNNC
- C14, C15: LCSC (none) -> CL10C200JB8NNNC
- R10, R9: LCSC (none) -> C125931
- R11: LCSC (none) -> C105578
- R8: LCSC (none) -> C227572
- U4: LCSC (none) -> C32843
- Y1: LCSC (none) -> C1985829
